File: pcb/switchnode.kicad_sch (KiCad schematic)
At the start: 5 parts, among them Q1 BC817, Q2 IRLML6402

Commit message: Rev2
Parts:
- removed R2: 10k, Resistor_SMD:R_0603_1608Metric, symbol Device:R
Connections:
- net +12V: now also Q2.2 (S); no longer Q2.3 (D)
- net SN_OUT: now also Q2.3 (D); no longer Q2.2 (S)
Other:
- moved on the sheet: Q1, R1, R29
