File: pcb/espio.kicad_sch (KiCad schematic)
At the start: 49 parts, among them J1 Conn_DEBUG, J2 Conn_I2C, P1 K776180WR-2, U1 MCP2562-E-SN, U4 NCV7805BDTRKG, U5 NCV8705MW33TCG

Commit message: Rev2
Parts:
- removed C3: 0.33uF, Capacitor_SMD:C_0603_1608Metric, symbol Device:C
- removed C5: 1uF, Capacitor_SMD:C_0603_1608Metric, symbol Device:C
- removed J1: Conn_DEBUG, Connector_PinHeader_2.54mm:PinHeader_1x04_P2.54mm_Vertical, symbol Connector_Generic:Conn_01x04
- removed J2: Conn_I2C, Connector_PinHeader_2.54mm:PinHeader_1x04_P2.54mm_Vertical, symbol Connector_Generic:Conn_01x04
- removed P1: K776180WR-2, lcsc:CONN-TH_35P-P4.00_K776180WR-2, symbol lcsc:K776180WR-2
- removed R68, R69, R70, R71: 2k7, Resistor_SMD:R_0603_1608Metric, symbol Device:R
- removed U4: NCV7805BDTRKG, lcsc:TO-252-2_L6.6-W6.1-P4.58-LS9.9-TL, symbol lcsc:NCV7805BDTRKG
- removed U5: NCV8705MW33TCG, lcsc:VDFN-8_L3.0-W3.0-P0.65-BL-EP, symbol lcsc:NCV8705MW33TCG
- added C3: RVT2A2R2M0605_C335981, lcsc:CAP-SMD_BD6.3-L6.6-W6.6-FD, symbol lcsc:RVT2A2R2M0605_C335981
- added D1: BZV55-B12,115, lcsc:SOD-80C_L3.3-W1.5-RD, symbol lcsc:BZV55-B12,115
- added JP3: Jumper_2_Open, Jumper:SolderJumper-2_P1.3mm_Open_Pad1.0x1.5mm, symbol Jumper:Jumper_2_Open
- added U5: LF50CPT-TR, lcsc:PPAK-5_L6.5-W6.1-P1.27-LS10.0-TL, symbol lcsc:LF50CPT-TR
- added U6: K776180WR-1, lcsc:CONN-TH_35P-P4.00_K776180WR-2, symbol lcsc:K776180WR-1
- C4: value 1uF -> 0.1uF
Connections:
- net I2C1_SCL is gone; now on net SwitchingNode5/SN_IN: U3.13 (38)
- net I2C1_SDA is gone; now on net SwitchingNode6/SN_IN: U3.12 (37)
- net +12V: now also C4.1, D1.1 (C), JP3.1 (A), U5.1 (VIN), U6.13, U6.24, U6.25
- net +3V3: no longer C4.1
- net +5V: now also C3.1, U5.5 (VOUT)
- net CAN_H: now also U6.21
- net CAN_L: now also U6.22
- net GND: now also C3.2, U5.3 (GND), U6.23, U6.34, U6.35
- net SwitchingNode1/SN_OUT: now also U6.12
- net SwitchingNode10/SN_IN: now also U3.5 (21); no longer U3.4 (20)
- net SwitchingNode10/SN_OUT: now also U6.3
- net SwitchingNode11/SN_IN: now also U3.4 (20); no longer U3.3 (19)
- net SwitchingNode11/SN_OUT: now also U6.2
- net SwitchingNode12/SN_OUT: now also U6.1
- net SwitchingNode2/SN_OUT: now also U6.11
- net SwitchingNode3/SN_OUT: now also U6.10
- net SwitchingNode4/SN_OUT: now also U6.9
- net SwitchingNode5/SN_IN: no longer U3.11 (36)
- net SwitchingNode5/SN_OUT: now also U6.8
- net SwitchingNode6/SN_IN: no longer U3.10 (35)
- net SwitchingNode6/SN_OUT: now also U6.7
- net SwitchingNode7/SN_IN: now also U3.11 (36); no longer U3.9 (0)
- net SwitchingNode7/SN_OUT: now also U6.6
- net SwitchingNode8/SN_IN: now also U3.10 (35); no longer U3.8 (45)
- net SwitchingNode8/SN_OUT: now also U6.5
- net SwitchingNode9/SN_IN: now also U3.8 (45); no longer U3.5 (21)
- net SwitchingNode9/SN_OUT: now also U6.4
- net IN_0 renamed I_14
- net I_14: now also U6.32
- net IN_1 renamed I_15
- net I_15: now also U6.33
- net IN_10 renamed I_8
- net I_8: now also U6.26
- net IN_11 renamed I_3
- net I_3: now also U6.16
- net IN_12 renamed I_4
- net I_4: now also U6.17
- net IN_13 renamed I_9
- net I_9: now also U6.27
- net IN_14 renamed I_10
- net I_10: now also U6.28
- net IN_2 renamed I_7
- net I_7: now also U6.20
- net IN_3 renamed I_6
- net I_6: now also U6.19
- net IN_4 renamed I_13
- net I_13: now also U6.31
- net IN_5 renamed I_5
- net I_5: now also U6.18
- net IN_6 renamed I_12
- net I_12: now also U6.30
- net IN_7 renamed I_11
- net I_11: now also U6.29
- net IN_8 renamed I_1
- net I_1: now also U6.14
- net IN_9 renamed I_2
- net I_2: now also U6.15
- net SN_IN_12: no longer names the net of U2.3 (14)
- new net: D1.2 (A), JP3.2 (B), U5.2 (INHIBIT)
- new net SwitchingNode12/SN_IN: U3.3 (19)
- no-connect marks 7 -> 6
Other:
- note added: "3V3 wird vom DevKit gemacht und nicht gebraucht."
- note removed: "Debug-Connector"

Commit message: working
Connections:
- net at U2.10 (3): now also R13.1, R14.2
- net SwitchingNode11/SN_IN: no longer names the net of U3.4 (20)
- new net OUT_12: U2.9 (46)
Changed lines of the file:
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@@
-	)
-	(junction
-		(at 97.79 128.27)
-		(diameter 0)
-		(color 0 0 0 0)
 	)
 	(junction
@@
 	)
 	(junction
+		(at 97.79 125.73)
+		(diameter 0)
+		(color 0 0 0 0)
+	)
+	(junction
 		(at 153.67 148.59)
 		(diameter 0)
@@
 	)
 	(no_connect
-		(at 125.73 125.73)
+		(at 153.67 140.97)
 	)
 	(no_connect
@@
 	(wire
 		(pts
+			(xy 97.79 125.73) (xy 97.79 148.59)
+		)
+		(stroke
+			(width 0)
+			(type default)
+		)
+	)
+	(wire
+		(pts
 			(xy 90.17 157.48) (xy 90.17 156.21)
 		)
@@
 	(wire
 		(pts
+			(xy 97.79 125.73) (xy 125.73 125.73)
+		)
+		(stroke
+			(width 0)
+			(type default)
+		)
+	)
+	(wire
+		(pts
 			(xy 95.25 93.98) (xy 95.25 130.81)
 		)
@@
 	(wire
 		(pts
-			(xy 97.79 148.59) (xy 97.79 128.27)
+			(xy 97.79 93.98) (xy 97.79 125.73)
 		)
 		(stroke
@@
 	(wire
 		(pts
-			(xy 175.26 140.97) (xy 175.26 168.91)
-		)
-		(stroke
-			(width 0)
-			(type default)
-		)
-	)
-	(wire
-		(pts
 			(xy 90.17 135.89) (xy 125.73 135.89)
 		)
@@
 	(wire
 		(pts
-			(xy 153.67 140.97) (xy 175.26 140.97)
-		)
-		(stroke
-			(width 0)
-			(type default)
-		)
-	)
-	(wire
-		(pts
-			(xy 97.79 93.98) (xy 97.79 128.27)
-		)
-		(stroke
-			(width 0)
-			(type default)
-		)
-	)
-	(wire
-		(pts
 			(xy 72.39 86.36) (xy 72.39 82.55)
 		)
@@
 	(wire
 		(pts
-			(xy 175.26 168.91) (xy 209.55 168.91)
-		)
-		(stroke
-			(width 0)
-			(type default)
-		)
-	)
-	(wire
-		(pts
 			(xy 237.49 138.43) (xy 256.54 138.43)
 		)
@@
 	(wire
 		(pts
-			(xy 97.79 128.27) (xy 125.73 128.27)
-		)
-		(stroke
-			(width 0)
-			(type default)
-		)
-	)
-	(wire
-		(pts
 			(xy 284.48 128.27) (xy 280.67 128.27)
 		)
@@
 		)
 	)
+	(global_label "OUT_12"
+		(shape input)
+		(at 209.55 168.91 180)
+		(fields_autoplaced yes)
+		(effects
+			(font
+				(size 1.27 1.27)
+			)
+			(justify right)
+		)
+		(property "Intersheetrefs" "${INTERSHEET_REFS}"
+			(at 199.5496 168.91 0)
+			(effects
+				(font
+					(size 1.27 1.27)
+				)
+				(justify right)
+				(hide yes)
+			)
+		)
+	)
 	(global_label "I_6"
 		(shape input)
@@
 				(hide yes)
 			)
+		)
+	)
+	(global_label "OUT_12"
+		(shape input)
+		(at 125.73 128.27 180)
+		(fields_autoplaced yes)
+		(effects
+			(font
+				(size 1.27 1.27)
+			)
+			(justify right)
+		)
+		(property "Intersheetrefs" "${INTERSHEET_REFS}"
+			(at 115.7296 128.27 0)
+			(effects
+				(font
+					(size 1.27 1.27)
+				)
+				(justify right)
+				(hide yes)
+			)

Commit message: some stuff
Parts:
- added J1: Conn_Dbg_Header, Connector_PinHeader_2.54mm:PinHeader_1x02_P2.54mm_Vertical_SMD_Pin1Left, symbol Connector_Generic:Conn_01x02
Connections:
- net CAN_H: now also J1.2 (Pin_2)
- net CAN_L: now also J1.1 (Pin_1)
Changed lines of the file:
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@@
 	(text "hier fehlt noch das\nüberspannungsdings\nOder anderer Transceiver?\nOder kann der das?"
 		(exclude_from_sim no)
-		(at 259.08 271.78 0)
+		(at 234.696 278.638 0)
 		(effects
 			(font
@@
 	(wire
 		(pts
+			(xy 275.59 248.92) (xy 275.59 265.43)
+		)
+		(stroke
+			(width 0)
+			(type default)
+		)
+	)
+	(wire
+		(pts
 			(xy 254 229.87) (xy 254 241.3)
 		)
@@
 	(wire
 		(pts
+			(xy 280.67 262.89) (xy 279.4 262.89)
+		)
+		(stroke
+			(width 0)
+			(type default)
+		)
+	)
+	(wire
+		(pts
 			(xy 237.49 168.91) (xy 264.16 168.91)
 		)
@@
 	(wire
 		(pts
+			(xy 279.4 254) (xy 279.4 262.89)
+		)
+		(stroke
+			(width 0)
+			(type default)
+		)
+	)
+	(wire
+		(pts
 			(xy 199.39 123.19) (xy 199.39 128.27)
 		)
@@
 	(wire
 		(pts
+			(xy 275.59 265.43) (xy 280.67 265.43)
+		)
+		(stroke
+			(width 0)
+			(type default)
+		)
+	)
+	(wire
+		(pts
 			(xy 85.09 140.97) (xy 85.09 148.59)
 		)
@@
 					(unit 1)
 				)
+			)
+		)
+	)
+	(symbol
+		(lib_id "Connector_Generic:Conn_01x02")
+		(at 285.75 262.89 0)
+		(unit 1)
+		(exclude_from_sim no)
+		(in_bom yes)
+		(on_board yes)
+		(dnp no)
+		(fields_autoplaced yes)
+		(property "Reference" "J1"
+			(at 288.29 262.8899 0)
+			(effects
+				(font
+					(size 1.27 1.27)
+				)
+				(justify left)
+			)
+		)
+		(property "Value" "Conn_Dbg_Header"
+			(at 288.29 265.4299 0)
+			(effects
+				(font
+					(size 1.27 1.27)
+				)
+				(justify left)
+			)
+		)
+		(property "Footprint" "Connector_PinHeader_2.54mm:PinHeader_1x02_P2.54mm_Vertical_SMD_Pin1Left"
+			(at 285.75 262.89 0)
+			(effects
+				(font
+					(size 1.27 1.27)
+				)
+				(hide yes)
+			)
+		)
+		(property "Datasheet" "~"
+			(at 285.75 262.89 0)
+			(effects
+				(font
+					(size 1.27 1.27)
+				)
+				(hide yes)
+			)
+		)
+		(property "Description" "Generic connector, single row, 01x02, script generated (kicad-library-utils/schlib/autogen/connector/)"
+			(at 285.75 262.89 0)
+			(effects
+				(font
+					(size 1.27 1.27)
+				)
+				(hide yes)
+			)
+		)
+		(pin "1"
+		)
+		(pin "2"
+		)
+		(instances
+			(project ""
+				(path "/b4b62778-ee22-463e-ba5d-5da015edb128"
+					(reference "J1")
+					(unit 1)
+				)

Commit message: safety commit
Parts:
- removed R33, R35, R37, R39, R41, R43, R45, R47: 33k, Resistor_SMD:R_0603_1608Metric, symbol Device:R
- removed R34, R36, R38, R40, R42, R44, R46, R48: 6k8, Resistor_SMD:R_0603_1608Metric, symbol Device:R
- added DSub1: 5007620481, lcsc:CONN-TH_5007620481, symbol lcsc:5007620481
- added Q10, Q11, Q12, Q13, Q14, Q15, Q9: BC817, Package_TO_SOT_SMD:SOT-23, symbol Transistor_BJT:BC817
- J1: footprint Connector_PinHeader_2.54mm:PinHeader_1x02_P2.54mm_Vertical_SMD_Pin1Left -> Connector_PinHeader_2.54mm:PinHeader_1x02_P2.54mm_Vertical
Connections:
- net I_11 is gone; now on net ABS_INPUT_HR_2: U6.29
- net I_12 is gone; now on net ABS_INPUT_HR_1: U6.30
- net I_13 is gone; now on net ABS_INPUT_HL_1: U6.31
- net I_14 is gone; now on net ABS_INPUT_VL_1: U6.32
- net I_15 is gone; now on net ABS_INPUT_VL_2: U6.33
- net I_5 is gone; now on net ABS_INPUT_HL_2: U6.18
- net I_6 is gone; now on net ABS_INPUT_VR_2: U6.19
- net I_7 is gone; now on net ABS_INPUT_VR_1: U6.20
- net SwitchingNode12/SN_OUT is gone; now on net OUT_1: U6.1
- net +12V: now also D1.2 (A); no longer D1.1 (C)
- net GND: now also DSub1.1, DSub1.2, Q10.2 (E), Q11.2 (E), Q12.2 (E), Q13.2 (E), Q14.2 (E), Q15.2 (E), Q9.2 (E)
- net ABS_INPUT_HR_2: now reaches U2.12 (18)
- net ABS_INPUT_HR_1: now reaches U2.13 (17)
- net ABS_INPUT_HL_2: now reaches U2.14 (16)
- net ABS_INPUT_HL_1: now reaches U2.15
- net ABS_INPUT_VR_2: now reaches U2.16 (8)
- net ABS_INPUT_VR_1: now reaches U2.17 (6)
- net ABS_INPUT_VL_2: now reaches U2.18 (5)
- net ABS_INPUT_VL_1: now reaches U2.19 (4)
- net at JP3.2 (B), U5.2 (INHIBIT): now also D1.1 (C); no longer D1.2 (A)
- net OUT_12 renamed OUT_1
- net SwitchingNode10/SN_IN: no longer names the net of U3.5 (21)
- net SwitchingNode10/SN_IN: now also Q13.1 (B)
- net SwitchingNode10/SN_OUT: no longer names the net of U6.3
- net SwitchingNode10/SN_OUT: now also Q13.3 (C)
- net SwitchingNode11/SN_OUT: no longer names the net of U6.2
- net SwitchingNode11/SN_OUT: now also Q14.3 (C)
- net SwitchingNode12/SN_IN: no longer names the net of U3.3 (19)
- net SwitchingNode12/SN_IN: now also Q14.1 (B)
- net SwitchingNode5/SN_IN: no longer names the net of U3.13 (38)
- net SwitchingNode5/SN_IN: now also Q11.1 (B)
- net SwitchingNode5/SN_OUT: no longer names the net of U6.8
- net SwitchingNode5/SN_OUT: now also Q11.3 (C)
- net SwitchingNode6/SN_IN: no longer names the net of U3.12 (37)
- net SwitchingNode6/SN_IN: now also Q9.1 (B)
- net SwitchingNode6/SN_OUT: no longer names the net of U6.7
- net SwitchingNode6/SN_OUT: now also Q9.3 (C)
- net SwitchingNode7/SN_IN: no longer names the net of U3.11 (36)
- net SwitchingNode7/SN_IN: now also Q10.1 (B)
- net SwitchingNode7/SN_OUT: no longer names the net of U6.6
- net SwitchingNode7/SN_OUT: now also Q10.3 (C)
- net SwitchingNode8/SN_IN: no longer names the net of U3.10 (35)
- net SwitchingNode8/SN_IN: now also Q15.1 (B)
- net SwitchingNode8/SN_OUT: no longer names the net of U6.5
- net SwitchingNode8/SN_OUT: now also Q15.3 (C)
- net SwitchingNode9/SN_IN: no longer names the net of U3.8 (45)
- net SwitchingNode9/SN_IN: now also Q12.1 (B)
- net SwitchingNode9/SN_OUT: no longer names the net of U6.4
- net SwitchingNode9/SN_OUT: now also Q12.3 (C)
Other:
- removed sheet SwitchingNode10
- removed sheet SwitchingNode11
- removed sheet SwitchingNode12
- removed sheet SwitchingNode5
- removed sheet SwitchingNode6
- removed sheet SwitchingNode7
- removed sheet SwitchingNode8
- removed sheet SwitchingNode9
- moved on the sheet: D1, J1, JP1, U6

Commit message: up to date
Parts:
- added J2: Conn_01x07, Connector_PinSocket_2.54mm:PinSocket_1x07_P2.54mm_Vertical, symbol Connector_Generic:Conn_01x07
- added J3: Conn_01x08, Connector_PinSocket_2.54mm:PinSocket_1x08_P2.54mm_Vertical, symbol Connector_Generic:Conn_01x08
- added JP2: VCC_as_Pin_8, Jumper:SolderJumper-2_P1.3mm_Open_Pad1.0x1.5mm, symbol Jumper:Jumper_2_Open
- Q14: lcsc (none) -> C52801
Connections:
- net +12V: now also JP2.1 (A)
- net ABS_INPUT_HL_1: now also J3.4 (Pin_4)
- net ABS_INPUT_HL_2: now also J3.3 (Pin_3)
- net ABS_INPUT_HR_1: now also J3.2 (Pin_2)
- net ABS_INPUT_HR_2: now also J3.1 (Pin_1)
- net ABS_INPUT_VL_1: now also J3.8 (Pin_8)
- net ABS_INPUT_VL_2: now also J3.7 (Pin_7)
- net ABS_INPUT_VR_1: now also J3.6 (Pin_6)
- net ABS_INPUT_VR_2: now also J3.5 (Pin_5)
- net I_1: now also JP2.2 (B)
- net at Q11.1 (B), U3.13 (38): now also J2.7 (Pin_7)
- net at Q13.1 (B), U3.5 (21): now also J2.2 (Pin_2)
- net at Q15.1 (B), U3.10 (35): now also J2.4 (Pin_4)
- net at Q9.1 (B), U3.12 (37): now also J2.6 (Pin_6)
- net at Q12.1 (B), U3.8 (45): now also J2.3 (Pin_3)
- net at Q10.1 (B), U3.11 (36): now also J2.5 (Pin_5)
- net at Q14.1 (B), U3.3 (19): now also J2.1 (Pin_1)
- net NC_RST: no longer names the net of U2.20 (RST)
- no-connect marks 6 -> 7
Other:
- moved on the sheet: Q11, Q12, Q13, Q14, Q15, Q9

Commit message: edited a lot
Parts:
- removed D1: BZV55-B12,115, lcsc:SOD-80C_L3.3-W1.5-RD, symbol lcsc:BZV55-B12,115
- added D2: BZV55C15_C545332, lcsc:SOD-80_L3.5-W1.5-RD, symbol lcsc:BZV55C15_C545332
- added J4: Conn_01x01, Connector_PinHeader_2.54mm:PinHeader_1x01_P2.54mm_Vertical, symbol Connector_Generic:Conn_01x01
- added Q16: BC817, Package_TO_SOT_SMD:SOT-23, symbol Transistor_BJT:BC817
- added R2: 4M, Resistor_SMD:R_0603_1608Metric, symbol Device:R
- added R3: 1M, Resistor_SMD:R_0603_1608Metric, symbol Device:R
Connections:
- net +12V: now also D2.1 (C), J4.1 (Pin_1), R2.1; no longer JP3.1 (A)
- net ABS_INPUT_HL_1: now also J3.5 (Pin_5), U2.16 (8), U6.19; no longer J3.4 (Pin_4), U2.15, U6.31
- net ABS_INPUT_VR_2: now also J3.4 (Pin_4), U2.15, U6.31; no longer J3.5 (Pin_5), U2.16 (8), U6.19
- net GND: now also JP3.1 (A), R3.2
- net at JP3.2 (B), U5.2 (INHIBIT): now also Q16.3 (C), R2.2
- net 8_PULL_DOWN: now reaches Q11.3 (C), U6.8
- net 3_PULL_DOWN: now reaches Q13.3 (C), U6.3
- net 5_PULL_DOWN: now reaches Q15.3 (C), U6.5
- net 7_PULL_DOWN: now reaches Q9.3 (C), U6.7
- net 4_PULL_DOWN: now reaches Q12.3 (C), U6.4
- net at J2.1 (Pin_1), Q14.1 (B): now also U3.4 (20); no longer U3.3 (19)
- net 6_PULL_DOWN: now reaches Q10.3 (C), U6.6
- net 2_PULL_DOWN: now reaches Q14.3 (C), U6.2
- net SwitchingNode1/SN_OUT renamed 12_12V_OUT
- net SwitchingNode2/SN_OUT renamed 11_12V_OUT
- net SwitchingNode3/SN_OUT renamed 10_12V_OUT
- net SwitchingNode4/SN_OUT renamed 9_12V_OUT
- new net: Q16.2 (E), R3.1
- new net: D2.2 (A), Q16.1 (B)
Other:
- note added: "Wenn Board in eingestecktem Zustand nicht einschaltet, muss vier auch unconnected bleiben."
- moved on the sheet: C4, JP3, U6

Commit message: Final stretch, maybe
Parts:
- removed Q14: BC817, Package_TO_SOT_SMD:SOT-23, symbol Transistor_BJT:BC817
- J2: footprint Connector_PinSocket_2.54mm:PinSocket_1x07_P2.54mm_Vertical -> Connector_PinSocket_2.54mm:PinSocket_1x06_P2.54mm_Vertical; symbol Connector_Generic:Conn_01x07 -> Connector_Generic:Conn_01x06
Connections:
- net at Q11.1 (B), U3.13 (38): now also J2.6 (Pin_6); no longer J2.7 (Pin_7)
- net at Q13.1 (B), U3.5 (21): now also J2.1 (Pin_1); no longer J2.2 (Pin_2)
- net at Q15.1 (B), U3.10 (35): now also J2.3 (Pin_3); no longer J2.4 (Pin_4)
- net at Q9.1 (B), U3.12 (37): now also J2.5 (Pin_5); no longer J2.6 (Pin_6)
- net at Q12.1 (B), U3.8 (45): now also J2.2 (Pin_2); no longer J2.3 (Pin_3)
- net at U3.4 (20): no longer J2.1 (Pin_1)
- net at Q10.1 (B), U3.11 (36): now also J2.4 (Pin_4); no longer J2.5 (Pin_5)
- net 2_PULL_DOWN: no longer names the net of U6.2
- no-connect marks 7 -> 9
Other:
- note removed: "Wenn Board in eingestecktem Zustand nicht einschaltet, muss vier auch unconnected bleiben."
