File: pcb/espio.kicad_sch (KiCad schematic)
At the start: 42 parts, among them J1 Conn_Dbg_Header, J2 Conn_01x07, J3 Conn_01x08, J4 Conn_01x01, Q10 BC817, Q11 BC817, Q12 BC817, Q13 BC817, Q15 BC817, Q16 BC817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

Commit message: Can-Thread-Split
Parts:
- removed DSub1: 5007620481, lcsc:CONN-TH_5007620481, symbol lcsc:5007620481

Commit message: fixed the dumb schematic
Parts:
- removed R13, R16, R50, R52, R54, R56, R58: 6k8, Resistor_SMD:R_0603_1608Metric, symbol Device:R
- removed R14, R15, R49, R51, R53, R55, R57: 33k, Resistor_SMD:R_0603_1608Metric, symbol Device:R
- added J5: Conn_01x08, Connector_PinSocket_2.54mm:PinSocket_1x08_P2.54mm_Vertical, symbol Connector_Generic:Conn_01x08
- added J6: Conn_01x08, Connector_PinSocket_2.54mm:PinSocket_1x04_P2.54mm_Vertical, symbol Connector_Generic:Conn_01x04
- added LED5: 0805G (Green), lcsc:LED0805-R-RD, symbol lcsc:0805G(Green)
- added R39: 470, Resistor_SMD:R_0603_1608Metric, symbol Device:R
- J1, J2, J3, J4: now left out of the parts list
- R2: value 4M -> 4k
- R3: value 1M -> 1k
Connections:
- net +5V: now also R39.1
- net GND: now also LED5.2 (K)
- net SwitchingNode1/SN_IN: now also J6.1 (Pin_1)
- net SwitchingNode2/SN_IN: now also J6.2 (Pin_2)
- net SwitchingNode3/SN_IN: now also J6.3 (Pin_3)
- net SwitchingNode4/SN_IN: now also J6.4 (Pin_4)
- net Spannungsteiler1/IN_MEAS: now reaches U2.4 (13)
- net Spannungsteiler1/IN_MEAS: now also J5.7 (Pin_7)
- net Spannungsteiler7/IN_MEAS: now reaches U2.10 (3)
- net Spannungsteiler7/IN_MEAS: now also J5.2 (Pin_2)
- net Spannungsteiler6/IN_MEAS: now reaches U2.11 (8)
- net Spannungsteiler6/IN_MEAS: now also J5.1 (Pin_1)
- net Spannungsteiler8/IN_MEAS: now reaches U2.3 (14)
- net Spannungsteiler8/IN_MEAS: now also J5.8 (Pin_8)
- net Spannungsteiler3/IN_MEAS: now reaches U2.5 (12)
- net Spannungsteiler3/IN_MEAS: now also J5.6 (Pin_6)
- net Spannungsteiler2/IN_MEAS: now reaches U2.6 (11)
- net Spannungsteiler2/IN_MEAS: now also J5.5 (Pin_5)
- net Spannungsteiler4/IN_MEAS: now reaches U2.7 (10)
- net Spannungsteiler4/IN_MEAS: now also J5.4 (Pin_4)
- net Spannungsteiler5/IN_MEAS: now reaches U2.8 (9)
- net Spannungsteiler5/IN_MEAS: now also J5.3 (Pin_3)
- net I_6: now reaches U6.2
- net OUT_1 renamed DIRECT_IN_1
- new net: LED5.1 (A), R39.2
- no-connect marks 8 -> 7
Other:
- added sheet Spannungsteiler1 (spannungsteiler.kicad_sch)
- added sheet Spannungsteiler2 (spannungsteiler.kicad_sch)
- added sheet Spannungsteiler3 (spannungsteiler.kicad_sch)
- added sheet Spannungsteiler4 (spannungsteiler.kicad_sch)
- added sheet Spannungsteiler5 (spannungsteiler.kicad_sch)
- added sheet Spannungsteiler6 (spannungsteiler.kicad_sch)
- added sheet Spannungsteiler7 (spannungsteiler.kicad_sch)
- added sheet Spannungsteiler8 (spannungsteiler.kicad_sch)
- moved on the sheet: C3, J2, J3, JP2, Q10, Q11, Q12, Q13, Q15, Q9, U2, U3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

Commit message: learned from my mistakes
Parts:
- removed Q10, Q11, Q12, Q13, Q15, Q9: BC817, Package_TO_SOT_SMD:SOT-23, symbol Transistor_BJT:BC817
- added D6: 1N5819HW-7-F, lcsc:SOD-123_L2.7-W1.6-LS3.7-RD, symbol lcsc:1N5819HW-7-F
- added F5: 1812L050/30PR, lcsc:F1812, symbol lcsc:1812L050_30PR
Connections:
- net I_10 is gone; now on net I_8: U6.28
- net +12V: now also D6.2 (A); no longer C4.1, U5.1 (VIN)
- net I_6: now also U6.26; no longer U6.2
- net I_8: no longer U6.26
- net pulldown6/IN: now reaches J2.6 (Pin_6), U3.13 (38)
- net pulldown1/IN: now reaches J2.1 (Pin_1), U3.5 (21)
- net pulldown3/IN: now reaches J2.3 (Pin_3), U3.10 (35)
- net pulldown5/IN: now reaches J2.5 (Pin_5), U3.12 (37)
- net pulldown2/IN: now reaches J2.2 (Pin_2), U3.8 (45)
- net pulldown4/IN: now reaches J2.4 (Pin_4), U3.11 (36)
- net I_9 renamed I_7
- new net: D6.1 (K), F5.1
- new net: C4.1, F5.2, U5.1 (VIN)
- new net I_5: U6.2
Other:
- added sheet pulldown1 (pulldown.kicad_sch)
- added sheet pulldown2 (pulldown.kicad_sch)
- added sheet pulldown3 (pulldown.kicad_sch)
- added sheet pulldown4 (pulldown.kicad_sch)
- added sheet pulldown5 (pulldown.kicad_sch)
- added sheet pulldown6 (pulldown.kicad_sch)
- sheet SwitchingNode1 ports: added POWER; removed none
- sheet SwitchingNode2 ports: added POWER; removed none
- sheet SwitchingNode3 ports: added POWER; removed none
- sheet SwitchingNode4 ports: added POWER; removed none
- note added: "- LED ist zu hell"
- moved on the sheet: C3, C4, D2, J2, J4, JP3, LED5, Q16, R2, R3, R39, U5
