File: pcb/espio.kicad_pcb (KiCad board)
At the start: 2 copper layers, 77.3 x 69.7 mm, 109 parts, among them J1 Conn_DEBUG, J2 Conn_I2C, P1 K776180WR-2, Q1 BC817, Q10 IRLML6402, Q11 BC817, Q12 IRLML6402, Q13 BC817, Q14 IRLML6402, Q15 BC817, Q16 IRLML6402, Q17 BC817, Q18 IRLML6402, Q19 BC817, Q2 IRLML6402, Q20 IRLML6402, Q21 BC817, Q22 IRLML6402, Q23 BC817, Q24 IRLML6402, Q3 BC817, Q4 IRLML6402, Q5 BC817, Q6 IRLML6402, Q7 BC817, Q8 IRLML6402, Q9 BC817, U1 MCP2562-E-SN, U4 NCV7805BDTRKG, U5 NCV8705MW33TCG

Commit message: Rev2
Parts:
- removed C5: 1uF, Capacitor_SMD:C_0603_1608Metric
- removed J1: Conn_DEBUG, Connector_PinHeader_2.54mm:PinHeader_1x04_P2.54mm_Vertical
- removed J2: Conn_I2C, Connector_PinHeader_2.54mm:PinHeader_1x04_P2.54mm_Vertical
- removed P1: K776180WR-2, lcsc:CONN-TH_35P-P4.00_K776180WR-2
- removed R10, R11, R12, R17, R2, R3, R4, R5, R6, R7, R8, R9: 10k, Resistor_SMD:R_0603_1608Metric
- removed R68, R69, R70, R71: 2k7, Resistor_SMD:R_0603_1608Metric
- removed U4: NCV7805BDTRKG, lcsc:TO-252-2_L6.6-W6.1-P4.58-LS9.9-TL
- added D1: BZV55-B12,115, lcsc:SOD-80C_L3.3-W1.5-RD, F.Cu at (114.0, 95.1)
- added JP3: Jumper_2_Open, Jumper:SolderJumper-2_P1.3mm_Open_Pad1.0x1.5mm, F.Cu at (115.2, 97.8)
- added U6: K776180WR-1, lcsc:CONN-TH_35P-P4.00_K776180WR-2, F.Cu at (139.6, 129.1)
- C3: value 0.33uF -> RVT2A2R2M0605_C335981; footprint Capacitor_SMD:C_0603_1608Metric -> lcsc:CAP-SMD_BD6.3-L6.6-W6.6-FD
- C4: value 1uF -> 0.1uF
- U5: value NCV8705MW33TCG -> LF50CPT-TR; footprint lcsc:VDFN-8_L3.0-W3.0-P0.65-BL-EP -> lcsc:PPAK-5_L6.5-W6.1-P1.27-LS10.0-TL
- moved C3 10.2 mm to (123.4, 90.4)
- moved C4 8.44 mm to (111.0, 91.2), turned to 90 degrees
- moved U5 0.69 mm to (115.1, 88.8), turned to 90 degrees
- moved C2 0.14 mm to (147.3, 91.9)
- turned Q10 to 90 degrees
- turned Q12 to 90 degrees
- turned Q14 to 90 degrees
- turned Q16 to 90 degrees
- turned Q18 to 90 degrees
- turned Q2 to 90 degrees
- turned Q20 to 90 degrees
- turned Q22 to 90 degrees
- turned Q24 to 90 degrees
- turned Q4 to 90 degrees
- turned Q6 to 90 degrees
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Connections:
- C3 pad 1: GND -> +5V
- C3 pad 2: +12V -> GND
- C4 pad 1: +3V3 -> +12V
- Q10 pad 2: /SwitchingNode5/SN_OUT -> +12V
- Q10 pad 3: +12V -> /SwitchingNode5/SN_OUT
- Q12 pad 2: /SwitchingNode6/SN_OUT -> +12V
- Q12 pad 3: +12V -> /SwitchingNode6/SN_OUT
- Q14 pad 2: /SwitchingNode7/SN_OUT -> +12V
- Q14 pad 3: +12V -> /SwitchingNode7/SN_OUT
- Q16 pad 2: /SwitchingNode8/SN_OUT -> +12V
- Q16 pad 3: +12V -> /SwitchingNode8/SN_OUT
- Q18 pad 2: /SwitchingNode9/SN_OUT -> +12V
- Q18 pad 3: +12V -> /SwitchingNode9/SN_OUT
- Q2 pad 2: /SwitchingNode1/SN_OUT -> +12V
- Q2 pad 3: +12V -> /SwitchingNode1/SN_OUT
- Q20 pad 2: /SwitchingNode10/SN_OUT -> +12V
- Q20 pad 3: +12V -> /SwitchingNode10/SN_OUT
- Q22 pad 2: /SwitchingNode11/SN_OUT -> +12V
- Q22 pad 3: +12V -> /SwitchingNode11/SN_OUT
- Q24 pad 2: /SwitchingNode12/SN_OUT -> +12V
- Q24 pad 3: +12V -> /SwitchingNode12/SN_OUT
- Q4 pad 2: /SwitchingNode2/SN_OUT -> +12V
- Q4 pad 3: +12V -> /SwitchingNode2/SN_OUT
- Q6 pad 2: /SwitchingNode3/SN_OUT -> +12V
- Q6 pad 3: +12V -> /SwitchingNode3/SN_OUT
- Q8 pad 2: /SwitchingNode4/SN_OUT -> +12V
- Q8 pad 3: +12V -> /SwitchingNode4/SN_OUT
- R14 pad 1: IN_13 -> I_9
- R15 pad 1: IN_14 -> I_10
- R28 pad 1: SN_IN_12 -> /SwitchingNode12/SN_IN
- R33 pad 1: IN_0 -> I_14
- R35 pad 1: IN_1 -> I_15
- R37 pad 1: IN_2 -> I_7
- R39 pad 1: IN_3 -> I_6
- R41 pad 1: IN_4 -> I_13
- R43 pad 1: IN_5 -> I_5
- R45 pad 1: IN_6 -> I_12
- R47 pad 1: IN_7 -> I_11
- R49 pad 1: IN_8 -> I_1
- R51 pad 1: IN_9 -> I_2
- R53 pad 1: IN_10 -> I_8
- R55 pad 1: IN_11 -> I_3
- R57 pad 1: IN_12 -> I_4
- U2 pad 3: SN_IN_12 -> unconnected-(U2-14-Pad3)
- U3 pad 10: /SwitchingNode6/SN_IN -> /SwitchingNode8/SN_IN
- U3 pad 11: /SwitchingNode5/SN_IN -> /SwitchingNode7/SN_IN
- U3 pad 12: I2C1_SDA -> /SwitchingNode6/SN_IN
- U3 pad 13: I2C1_SCL -> /SwitchingNode5/SN_IN
- U3 pad 3: /SwitchingNode11/SN_IN -> /SwitchingNode12/SN_IN
- U3 pad 4: /SwitchingNode10/SN_IN -> /SwitchingNode11/SN_IN
- U3 pad 5: /SwitchingNode9/SN_IN -> /SwitchingNode10/SN_IN
- U3 pad 8: /SwitchingNode8/SN_IN -> /SwitchingNode9/SN_IN
- U3 pad 9: /SwitchingNode7/SN_IN -> unconnected-(U3-0-Pad9)
- U5 pad 1: +3V3 -> +12V
- U5 pad 2: unconnected-(U5-N/C-Pad2) -> Net-(D1-A)
- U5 pad 3: unconnected-(U5-N/C-Pad3) -> GND
- U5 pad 4: GND -> unconnected-(U5-NC-Pad4)
- U5 pad 5: +3V3 -> +5V
Routing:
- net I_11: track 0.00 -> 125.6 mm, vias 0 -> 1
- net IN_7: track 125.6 -> 0.00 mm, vias 1 -> 0
- net I_5: track 0.00 -> 118.2 mm
- net IN_5: track 118.2 -> 0.00 mm
- net I_12: track 0.00 -> 117.6 mm
- net IN_6: track 117.6 -> 0.00 mm
- net I_10: track 0.00 -> 117.0 mm, vias 0 -> 1
- net IN_14: track 117.0 -> 0.00 mm, vias 1 -> 0
- net I_4: track 0.00 -> 110.9 mm, vias 0 -> 1
- net IN_12: track 110.9 -> 0.00 mm, vias 1 -> 0
- net I_3: track 0.00 -> 107.9 mm
- net IN_11: track 107.4 -> 0.00 mm
- net I_9: track 0.00 -> 106.5 mm, vias 0 -> 1
- net IN_13: track 106.5 -> 0.00 mm, vias 1 -> 0
- net I_13: track 0.00 -> 104.8 mm
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Other:
- board text added: "GND GND"
- board text added: "Permanent_On"
- board text removed: "I2C_0 I2C_1"
- board text removed: "SCL SDA SCL SDA"

Commit message: working
Parts:
- moved R13 2.54 mm to (136.8, 82.4)
- moved R14 2.54 mm to (136.8, 75.6)
Connections:
- R13 pad 1: Net-(U2-46) -> Net-(U2-3)
- R14 pad 2: Net-(U2-46) -> Net-(U2-3)
- R27 pad 1: /SwitchingNode11/SN_IN -> OUT_12
- U2 pad 10: unconnected-(U2-3-Pad10) -> Net-(U2-3)
- U2 pad 9: Net-(U2-46) -> OUT_12
- U3 pad 4: /SwitchingNode11/SN_IN -> unconnected-(U3-20-Pad4)
Routing:
- net OUT_12: track 0.00 -> 35.1 mm, vias 0 -> 1
- net Net-(U2-46): track 5.21 -> 0.00 mm
- net Net-(U2-3): track 0.00 -> 5.21 mm
- net /SwitchingNode11/SN_IN: track 3.32 -> 0.00 mm
- net I_9: track 106.5 -> 109.6 mm
- net unconnected-(U3-20-Pad4): track 0.00 -> 0.56 mm
Other:
- board text added: "rev2"
- board text removed: "GND RST 5V 12V"

Commit message: safety commit
Parts:
- removed Q16, Q18, Q20, Q22, Q24: IRLML6402, Package_TO_SOT_SMD:SOT-23
- removed Q17, Q19, Q21, Q23: BC817, Package_TO_SOT_SMD:SOT-23
- removed R21, R22, R23, R24, R25, R26, R27, R28: 100R, Resistor_SMD:R_0603_1608Metric
- removed R33, R35, R37, R39, R41, R43, R45, R47: 33k, Resistor_SMD:R_0603_1608Metric
- removed R34, R36, R38, R40, R42, R44, R46, R48: 6k8, Resistor_SMD:R_0603_1608Metric
- removed R59, R60, R61, R62, R64, R65, R66, R67: 10k, Resistor_SMD:R_0603_1608Metric
- added DSub1: 5007620481, lcsc:CONN-TH_5007620481, F.Cu at (244.6, 111.3)
- added J1: Conn_Dbg_Header, Connector_PinHeader_2.54mm:PinHeader_1x02_P2.54mm_Vertical, F.Cu at (164.8, 97.3)
- Q10, Q12, Q14: value IRLML6402 -> BC817
- moved Q14 17.0 mm to (121.7, 120.2), turned to -90 degrees
- moved Q13 14.5 mm to (125.5, 120.3)
- moved Q12 13.2 mm to (129.5, 120.5), turned to -90 degrees
- moved Q11 10.0 mm to (145.5, 120.5)
- moved Q9 9.72 mm to (141.5, 120.5)
- moved Q10 9.10 mm to (137.7, 120.5), turned to -90 degrees
- moved Q15 9.02 mm to (133.6, 120.5)
- moved C1 3.61 mm to (156.2, 95.5)
- turned D1 to 180 degrees
Connections:
- D1 pad 1: +12V -> Net-(D1-C)
- D1 pad 2: Net-(D1-A) -> +12V
- JP3 pad 2: Net-(D1-A) -> Net-(D1-C)
- Q10 pad 1: Net-(Q10-G) -> Net-(Q10-B)
- Q10 pad 2: +12V -> GND
- Q10 pad 3: /SwitchingNode5/SN_OUT -> Net-(Q10-C)
- Q12 pad 1: Net-(Q11-C) -> Net-(Q12-B)
- Q12 pad 2: +12V -> GND
- Q12 pad 3: /SwitchingNode6/SN_OUT -> Net-(Q12-C)
- Q14 pad 1: Net-(Q13-C) -> Net-(Q14-B)
- Q14 pad 2: +12V -> GND
- Q14 pad 3: /SwitchingNode7/SN_OUT -> Net-(Q14-C)
- Q9 pad 3: Net-(Q10-G) -> Net-(Q9-C)
- U2 pad 12: Net-(U2-18) -> ABS_INPUT_HR_2
- U2 pad 13: Net-(U2-17) -> ABS_INPUT_HR_1
- U2 pad 14: Net-(U2-16) -> ABS_INPUT_HL_2
- U2 pad 15: Net-(R41-Pad2) -> ABS_INPUT_HL_1
- U2 pad 16: Net-(R39-Pad2) -> ABS_INPUT_VR_2
- U2 pad 17: Net-(U2-6) -> ABS_INPUT_VR_1
- U2 pad 18: Net-(U2-5) -> ABS_INPUT_VL_2
- U2 pad 19: Net-(U2-4) -> ABS_INPUT_VL_1
- U2 pad 9: OUT_12 -> OUT_1
- U3 pad 10: /SwitchingNode8/SN_IN -> Net-(Q15-B)
- U3 pad 11: /SwitchingNode7/SN_IN -> Net-(Q10-B)
- U3 pad 12: /SwitchingNode6/SN_IN -> Net-(Q9-B)
- U3 pad 13: /SwitchingNode5/SN_IN -> Net-(Q11-B)
- U3 pad 3: /SwitchingNode12/SN_IN -> Net-(Q14-B)
- U3 pad 5: /SwitchingNode10/SN_IN -> Net-(Q13-B)
- U3 pad 8: /SwitchingNode9/SN_IN -> Net-(Q12-B)
- U5 pad 2: Net-(D1-A) -> Net-(D1-C)
- U6 pad 1: /SwitchingNode12/SN_OUT -> OUT_1
- U6 pad 18: I_5 -> ABS_INPUT_HL_2
- U6 pad 19: I_6 -> ABS_INPUT_VR_2
- U6 pad 2: /SwitchingNode11/SN_OUT -> Net-(Q14-C)
- U6 pad 20: I_7 -> ABS_INPUT_VR_1
- U6 pad 29: I_11 -> ABS_INPUT_HR_2
- U6 pad 3: /SwitchingNode10/SN_OUT -> Net-(Q13-C)
- U6 pad 30: I_12 -> ABS_INPUT_HR_1
- U6 pad 31: I_13 -> ABS_INPUT_HL_1
- U6 pad 32: I_14 -> ABS_INPUT_VL_1
- U6 pad 33: I_15 -> ABS_INPUT_VL_2
- U6 pad 4: /SwitchingNode9/SN_OUT -> Net-(Q12-C)
- U6 pad 5: /SwitchingNode8/SN_OUT -> Net-(Q15-C)
- U6 pad 6: /SwitchingNode7/SN_OUT -> Net-(Q10-C)
- U6 pad 7: /SwitchingNode6/SN_OUT -> Net-(Q9-C)
- U6 pad 8: /SwitchingNode5/SN_OUT -> Net-(Q11-C)
Routing:
- net ABS_INPUT_HR_2: track 0.00 -> 129.4 mm
- net I_11: track 125.6 -> 0.00 mm, vias 1 -> 0
- net I_5: track 118.2 -> 0.00 mm
- net I_12: track 117.6 -> 0.00 mm
- net ABS_INPUT_HL_2: track 0.00 -> 116.1 mm
- net ABS_INPUT_HR_1: track 0.00 -> 115.8 mm
- net I_13: track 104.8 -> 0.00 mm
- net ABS_INPUT_HL_1: track 0.00 -> 103.0 mm
- net I_6: track 99.0 -> 0.00 mm, vias 1 -> 0
- net ABS_INPUT_VR_2: track 0.00 -> 96.5 mm
- net I_7: track 90.6 -> 0.00 mm, vias 1 -> 0
- net ABS_INPUT_VR_1: track 0.00 -> 88.0 mm
- net +12V: track 172.7 -> 86.4 mm, vias 12 -> 4
- net I_15: track 79.5 -> 0.00 mm
- net ABS_INPUT_VL_2: track 0.00 -> 79.2 mm
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Other:
- board size 77.3 x 69.7 mm -> 191.4 x 118.2 mm

Commit message: up to date
Parts:
- removed DSub1: 5007620481, lcsc:CONN-TH_5007620481
- added J2: Conn_01x07, Connector_PinSocket_2.54mm:PinSocket_1x07_P2.54mm_Vertical, F.Cu at (130.1, 111.5)
- added J3: Conn_01x08, Connector_PinSocket_2.54mm:PinSocket_1x08_P2.54mm_Vertical, F.Cu at (142.5, 82.8)
- added JP2: VCC_as_Pin_8, Jumper:SolderJumper-2_P1.3mm_Open_Pad1.0x1.5mm, F.Cu at (111.0, 114.4)
- moved C1 2.05 mm to (154.2, 95.5), turned to 180 degrees
- moved J1 1.48 mm to (163.6, 96.5), turned to 0 degrees
Connections:
- U2 pad 20: NC_RST -> unconnected-(U2-RST-Pad20)
Routing:
- net Net-(J2-Pin_1): track 16.8 -> 28.0 mm
- net Net-(J2-Pin_2): track 16.0 -> 23.7 mm
- net ABS_INPUT_HR_1: track 115.8 -> 120.0 mm
- net ABS_INPUT_VL_2: track 79.2 -> 83.2 mm
- net ABS_INPUT_HR_2: track 129.4 -> 133.4 mm
- net ABS_INPUT_HL_2: track 116.1 -> 120.2 mm
- net ABS_INPUT_VR_2: track 96.5 -> 100.6 mm
- net ABS_INPUT_VL_1: track 79.1 -> 83.1 mm
- net ABS_INPUT_HL_1: track 103.0 -> 107.1 mm
- net ABS_INPUT_VR_1: track 88.0 -> 92.1 mm
- net CAN_H: track 61.0 -> 63.9 mm
- net Net-(J2-Pin_3): track 15.9 -> 18.8 mm
- net I_1: track 78.0 -> 79.8 mm
- net Net-(J2-Pin_6): track 16.0 -> 17.1 mm
- net CAN_L: track 56.0 -> 57.0 mm
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Other:
- board size 191.4 x 118.2 mm -> 77.3 x 69.7 mm
- board text added: "CAN_L CAN_H"

Commit message: edited a lot
Parts:
- removed D1: BZV55-B12,115, lcsc:SOD-80C_L3.3-W1.5-RD
- added D2: BZV55C15_C545332, lcsc:SOD-80_L3.5-W1.5-RD, F.Cu at (115.8, 96.0)
- added J4: Conn_01x01, Connector_PinHeader_2.54mm:PinHeader_1x01_P2.54mm_Vertical, F.Cu at (112.8, 99.3)
- added Q16: BC817, Package_TO_SOT_SMD:SOT-23, F.Cu at (120.1, 98.6)
- added R2: 4M, Resistor_SMD:R_0603_1608Metric, F.Cu at (116.5, 98.0)
- added R3: 1M, Resistor_SMD:R_0603_1608Metric, F.Cu at (116.5, 99.8)
- moved JP3 6.25 mm to (120.9, 95.2), turned to 180 degrees
- moved C3 1.78 mm to (123.4, 88.6)
Connections:
- net /SwitchingNode1/SN_OUT renamed /12_12V_OUT
- net /SwitchingNode2/SN_OUT renamed /11_12V_OUT
- net /SwitchingNode3/SN_OUT renamed /10_12V_OUT
- net /SwitchingNode4/SN_OUT renamed /9_12V_OUT
- net Net-(Q10-C) renamed /6_PULL_DOWN
- net Net-(Q11-C) renamed /8_PULL_DOWN
- net Net-(Q12-C) renamed /4_PULL_DOWN
- net Net-(Q13-C) renamed /3_PULL_DOWN
- net Net-(Q14-C) renamed /2_PULL_DOWN
- net Net-(Q15-C) renamed /5_PULL_DOWN
- net Net-(Q9-C) renamed /7_PULL_DOWN
- J3 pad 4: ABS_INPUT_HL_1 -> ABS_INPUT_VR_2
- J3 pad 5: ABS_INPUT_VR_2 -> ABS_INPUT_HL_1
- JP3 pad 1: +12V -> GND
- U2 pad 15: ABS_INPUT_HL_1 -> ABS_INPUT_VR_2
- U2 pad 16: ABS_INPUT_VR_2 -> ABS_INPUT_HL_1
- U3 pad 3: Net-(J2-Pin_1) -> unconnected-(U3-19-Pad3)
- U3 pad 4: unconnected-(U3-20-Pad4) -> Net-(J2-Pin_1)
- U6 pad 19: ABS_INPUT_VR_2 -> ABS_INPUT_HL_1
- U6 pad 31: ABS_INPUT_HL_1 -> ABS_INPUT_VR_2
Routing:
- net +12V: track 86.2 -> 100.4 mm
- net Net-(JP3-B): track 6.41 -> 15.3 mm
- net ABS_INPUT_VR_2: track 100.6 -> 107.1 mm
- net ABS_INPUT_HL_1: track 107.1 -> 100.6 mm
- net Net-(D2-A): track 0.00 -> 2.69 mm
- net Net-(J2-Pin_1): track 28.0 -> 25.4 mm
- net Net-(Q16-E): track 0.00 -> 2.00 mm
- net +5V: track 48.5 -> 47.6 mm
- net unconnected-(U3-20-Pad4): track 0.56 -> 0.00 mm
Other:
- board text added: "rev3"
- board text removed: "rev2"

Commit message: recovered lost pcb
Parts:
- removed Q14: BC817, Package_TO_SOT_SMD:SOT-23
- removed R49, R51, R53, R55, R57: 33k, Resistor_SMD:R_0603_1608Metric
- removed R50, R52, R54, R56, R58: 6k8, Resistor_SMD:R_0603_1608Metric
- added J6: Conn_01x08, Connector_PinSocket_2.54mm:PinSocket_1x04_P2.54mm_Vertical, F.Cu at (154.4, 94.6)
- added LED1: 0805G (Green), lcsc:LED0805-R-RD, F.Cu at (165.9, 110.0)
- added LED2: 0805G (Green), lcsc:LED0805-R-RD, F.Cu at (159.3, 110.0)
- added LED3: 0805G (Green), lcsc:LED0805-R-RD, F.Cu at (152.7, 110.0)
- added LED4: 0805G (Green), lcsc:LED0805-R-RD, F.Cu at (146.3, 110.0)
- added LED5: 0805G (Green), lcsc:LED0805-R-RD, F.Cu at (110.2, 80.8)
- added R10: DNP, Resistor_THT:R_Axial_DIN0207_L6.3mm_D2.5mm_P7.62mm_Horizontal, F.Cu at (149.1, 121.4)
- added R11: DNP, Resistor_THT:R_Axial_DIN0207_L6.3mm_D2.5mm_P7.62mm_Horizontal, F.Cu at (142.5, 121.4)
- added R12: 3k, Resistor_SMD:R_0603_1608Metric, F.Cu at (106.2, 102.1)
- added R17: 750R, Resistor_SMD:R_0603_1608Metric, F.Cu at (125.2, 76.5)
- added R21: 3k, Resistor_SMD:R_0603_1608Metric, F.Cu at (108.2, 102.1)
- added R22: 750R, Resistor_SMD:R_0603_1608Metric, F.Cu at (122.2, 76.5)
- added R23: 3k, Resistor_SMD:R_0603_1608Metric, F.Cu at (107.2, 105.4)
- added R24: 750R, Resistor_SMD:R_0603_1608Metric, F.Cu at (123.7, 76.5)
- added R25: 3k, Resistor_SMD:R_0603_1608Metric, F.Cu at (105.2, 105.4)
- added R26: 750R, Resistor_SMD:R_0603_1608Metric, F.Cu at (126.7, 76.5)
- added R27: 3k, Resistor_SMD:R_0603_1608Metric, F.Cu at (110.2, 102.1)
- added R28: 750R, Resistor_SMD:R_0603_1608Metric, F.Cu at (128.3, 76.5)
- added R33: 3k, Resistor_SMD:R_0603_1608Metric, F.Cu at (103.4, 105.4)
- added R34: 750R, Resistor_SMD:R_0603_1608Metric, F.Cu at (138.2, 76.5)
- added R35: 3k, Resistor_SMD:R_0603_1608Metric, F.Cu at (104.1, 102.1)
- added R36: 750R, Resistor_SMD:R_0603_1608Metric, F.Cu at (136.7, 76.5)
- added R37: 2k4, Resistor_SMD:R_0603_1608Metric, F.Cu at (153.2, 106.2)
- added R38: 2k4, Resistor_SMD:R_0603_1608Metric, F.Cu at (146.8, 106.2)
- added R39: 470, Resistor_SMD:R_0603_1608Metric, F.Cu at (110.2, 77.0)
- added R4: DNP, Resistor_THT:R_Axial_DIN0207_L6.3mm_D2.5mm_P7.62mm_Horizontal, F.Cu at (165.6, 121.4)
- added R5: DNP, Resistor_THT:R_Axial_DIN0207_L6.3mm_D2.5mm_P7.62mm_Horizontal, F.Cu at (159.0, 121.4)
- added R6: DNP, Resistor_THT:R_Axial_DIN0207_L6.3mm_D2.5mm_P7.62mm_Horizontal, F.Cu at (152.4, 121.4)
- added R7: DNP, Resistor_THT:R_Axial_DIN0207_L6.3mm_D2.5mm_P7.62mm_Horizontal, F.Cu at (145.8, 121.4)
- added R8: DNP, Resistor_THT:R_Axial_DIN0207_L6.3mm_D2.5mm_P7.62mm_Horizontal, F.Cu at (162.3, 121.4)
- added R9: DNP, Resistor_THT:R_Axial_DIN0207_L6.3mm_D2.5mm_P7.62mm_Horizontal, F.Cu at (155.7, 121.4)
- J2: footprint Connector_PinSocket_2.54mm:PinSocket_1x07_P2.54mm_Vertical -> Connector_PinSocket_2.54mm:PinSocket_1x06_P2.54mm_Vertical
- R1, R18, R19, R20: value 100R -> 1k
- R13, R16: value 6k8 -> 2k4
- R14: value 33k -> 3k
- R15: value 33k -> 750R
- R2: value 4M -> 4k
- R3: value 1M -> 1k
- moved R14 40.6 mm to (109.2, 105.4), turned to 90 degrees
- moved R13 38.0 mm to (166.4, 106.2), turned to 90 degrees
- moved R16 31.4 mm to (159.8, 106.2), turned to 90 degrees
- moved R15 18.7 mm to (120.7, 76.5)
- moved R32 13.9 mm to (143.5, 102.9), turned to 90 degrees
- moved R31 13.3 mm to (149.9, 102.6), turned to 90 degrees
- moved R30 12.9 mm to (156.5, 102.4), turned to 90 degrees
- moved R29 12.4 mm to (162.6, 102.6), turned to 90 degrees
- moved Q8 12.3 mm to (143.3, 110.5), turned to -90 degrees
- moved Q6 11.2 mm to (149.6, 110.3), turned to -90 degrees
- moved Q4 10.6 mm to (156.3, 110.0), turned to -90 degrees
- moved Q2 10.1 mm to (162.6, 110.2), turned to -90 degrees
- moved Q11 7.54 mm to (138.2, 118.9)
- moved Q9 7.27 mm to (135.9, 115.8)
- moved R20 7.16 mm to (145.0, 102.9)
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Connections:
- Q10 pad 1: Net-(J2-Pin_5) -> Net-(J2-Pin_4)
- Q11 pad 1: Net-(J2-Pin_7) -> Net-(J2-Pin_6)
- Q12 pad 1: Net-(J2-Pin_3) -> Net-(J2-Pin_2)
- Q13 pad 1: Net-(J2-Pin_2) -> Net-(J2-Pin_1)
- Q15 pad 1: Net-(J2-Pin_4) -> Net-(J2-Pin_3)
- Q2 pad 3: /12_12V_OUT -> Net-(Q2-D)
- Q4 pad 3: /11_12V_OUT -> Net-(Q4-D)
- Q6 pad 3: /10_12V_OUT -> Net-(Q6-D)
- Q8 pad 3: /9_12V_OUT -> Net-(Q8-D)
- Q9 pad 1: Net-(J2-Pin_6) -> Net-(J2-Pin_5)
- R13 pad 1: Net-(U2-3) -> Net-(LED1-A)
- R13 pad 2: GND -> Net-(Q2-D)
- R14 pad 1: I_9 -> I_6
- R14 pad 2: Net-(U2-3) -> /Spannungsteiler8/IN_MEAS
- R15 pad 1: I_10 -> /Spannungsteiler8/IN_MEAS
- R15 pad 2: Net-(R15-Pad2) -> GND
- R16 pad 1: Net-(R15-Pad2) -> Net-(LED2-A)
- R16 pad 2: GND -> Net-(Q4-D)
- U2 pad 10: Net-(U2-3) -> /Spannungsteiler7/IN_MEAS
- U2 pad 11: Net-(R15-Pad2) -> /Spannungsteiler6/IN_MEAS
- U2 pad 3: unconnected-(U2-14-Pad3) -> /Spannungsteiler8/IN_MEAS
- U2 pad 4: Net-(U2-13) -> /Spannungsteiler1/IN_MEAS
- U2 pad 5: Net-(U2-12) -> /Spannungsteiler3/IN_MEAS
- U2 pad 6: Net-(U2-11) -> /Spannungsteiler2/IN_MEAS
- U2 pad 7: Net-(U2-10) -> /Spannungsteiler4/IN_MEAS
- U2 pad 8: Net-(U2-9) -> /Spannungsteiler5/IN_MEAS
- U3 pad 10: Net-(J2-Pin_4) -> Net-(J2-Pin_3)
- U3 pad 11: Net-(J2-Pin_5) -> Net-(J2-Pin_4)
- U3 pad 12: Net-(J2-Pin_6) -> Net-(J2-Pin_5)
- U3 pad 13: Net-(J2-Pin_7) -> Net-(J2-Pin_6)
- U3 pad 4: Net-(J2-Pin_1) -> unconnected-(U3-20-Pad4)
- U3 pad 5: Net-(J2-Pin_2) -> Net-(J2-Pin_1)
- U3 pad 8: Net-(J2-Pin_3) -> Net-(J2-Pin_2)
- U6 pad 2: /2_PULL_DOWN -> I_6
Routing:
- net /Spannungsteiler6/IN_MEAS: track 0.00 -> 69.4 mm, vias 0 -> 1
- net /Spannungsteiler7/IN_MEAS: track 0.00 -> 62.0 mm, vias 0 -> 1
- net /Spannungsteiler4/IN_MEAS: track 0.00 -> 59.5 mm
- net I_9: track 109.6 -> 51.4 mm
- net /Spannungsteiler5/IN_MEAS: track 0.00 -> 57.4 mm, vias 0 -> 1
- net I_10: track 117.0 -> 59.9 mm
- net /Spannungsteiler2/IN_MEAS: track 0.00 -> 52.1 mm
- net I_3: track 107.9 -> 56.0 mm
- net /Spannungsteiler3/IN_MEAS: track 0.00 -> 51.3 mm
- net I_4: track 110.9 -> 63.0 mm
- net I_8: track 95.9 -> 48.8 mm
- net I_2: track 86.4 -> 41.7 mm
- net /Spannungsteiler8/IN_MEAS: track 0.00 -> 44.5 mm
- net /Spannungsteiler1/IN_MEAS: track 0.00 -> 44.5 mm
- net I_1: track 79.8 -> 39.3 mm
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Other:
- board size 77.3 x 69.7 mm -> 77.1 x 69.7 mm
- board text added: "3V3"
- board text added: "rev2.5"
- board text removed: "GND GND"
- board text removed: "rev3"

Commit message: learned from my mistakes
Parts:
- removed R4, R5, R6, R7: DNP, Resistor_THT:R_Axial_DIN0207_L6.3mm_D2.5mm_P7.62mm_Horizontal
- added D1: 1N5819HW-7-F, lcsc:SOD-123_L2.7-W1.6-LS3.7-RD, F.Cu at (121.0, 73.7)
- added D3: 1N5819HW-7-F, lcsc:SOD-123_L2.7-W1.6-LS3.7-RD, F.Cu at (121.0, 56.8)
- added D4: 1N5819HW-7-F, lcsc:SOD-123_L2.7-W1.6-LS3.7-RD, F.Cu at (95.1, 69.6)
- added D5: 1N5819HW-7-F, lcsc:SOD-123_L2.7-W1.6-LS3.7-RD, F.Cu at (121.0, 39.9)
- added D6: 1N5819HW-7-F, lcsc:SOD-123_L2.7-W1.6-LS3.7-RD, F.Cu at (103.4, 45.6)
- added F1: 1812L110/33MR, lcsc:F1812, F.Cu at (120.3, 63.2)
- added F2: 1812L110/33MR, lcsc:F1812, F.Cu at (120.3, 46.3)
- added F3: 1812L110/33MR, lcsc:F1812, F.Cu at (94.4, 59.2)
- added F4: 1812L110/33MR, lcsc:F1812, F.Cu at (120.3, 29.4)
- added F5: 1812L050/30PR, lcsc:F1812, F.Cu at (90.4, 51.8)
- added J5: Conn_01x08, Connector_PinSocket_2.54mm:PinSocket_1x08_P2.54mm_Vertical, F.Cu at (94.0, 29.1)
- moved Q9 100.7 mm to (84.6, 29.2), turned to 0 degrees
- moved Q10 98.1 mm to (84.6, 33.8), turned to 0 degrees
- moved Q11 96.6 mm to (84.6, 38.5), turned to 0 degrees
- moved R11 89.5 mm to (114.5, 36.4), turned to 0 degrees
- moved Q12 87.9 mm to (84.6, 43.1), turned to 0 degrees
- moved J2 85.2 mm to (98.6, 29.1), turned to 0 degrees
- moved Q7 84.4 mm to (110.5, 29.2), turned to 0 degrees
- moved Q8 83.4 mm to (110.5, 33.8), turned to 0 degrees
- moved J6 83.2 mm to (103.2, 29.1), turned to 0 degrees
- moved R10 82.0 mm to (88.6, 66.1), turned to 0 degrees
- moved Q5 81.2 mm to (84.6, 59.0), turned to 0 degrees
- moved R20 80.6 mm to (114.9, 28.1), turned to 0 degrees
- moved Q6 80.1 mm to (84.6, 63.6), turned to 0 degrees
- moved Q13 80.0 mm to (84.6, 47.7), turned to 0 degrees
- moved R38 79.7 mm to (114.9, 33.1), turned to 0 degrees
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Connections:
- net OUT_1 renamed DIRECT_IN_1
- C4 pad 1: +12V -> Net-(U5-VIN)
- Q2 pad 2: +12V -> Net-(Q2-S)
- Q4 pad 2: +12V -> Net-(Q4-S)
- Q6 pad 2: +12V -> Net-(Q6-S)
- Q8 pad 2: +12V -> Net-(Q8-S)
- R10 pad 1: /10_12V_OUT -> Net-(D4-A)
- R11 pad 1: /9_12V_OUT -> Net-(D5-A)
- R8 pad 1: /12_12V_OUT -> Net-(D1-A)
- R9 pad 1: /11_12V_OUT -> Net-(D3-A)
- U5 pad 1: +12V -> Net-(U5-VIN)
Routing:
- net ABS_INPUT_HR_2: track 132.7 -> 0.00 mm
- net ABS_INPUT_HL_2: track 124.4 -> 0.00 mm
- net ABS_INPUT_HR_1: track 124.1 -> 0.00 mm
- net ABS_INPUT_VR_2: track 111.3 -> 0.00 mm
- net ABS_INPUT_HL_1: track 106.7 -> 0.00 mm
- net ABS_INPUT_VR_1: track 98.7 -> 0.00 mm
- net +12V: track 112.1 -> 27.7 mm, vias 4 -> 0
- net ABS_INPUT_VL_2: track 83.5 -> 0.00 mm
- net ABS_INPUT_VL_1: track 79.6 -> 0.00 mm
- net /Spannungsteiler6/IN_MEAS: track 69.4 -> 0.00 mm, vias 1 -> 0
- net I_4: track 63.0 -> 0.00 mm, vias 1 -> 0
- net CAN_H: track 70.5 -> 7.88 mm
- net /Spannungsteiler7/IN_MEAS: track 62.0 -> 0.00 mm, vias 1 -> 0
- net DIRECT_IN_1: track 60.0 -> 0.00 mm, vias 1 -> 0
- net I_10: track 59.9 -> 0.00 mm, vias 1 -> 0
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Other:
- board size 77.1 x 69.7 mm -> 77.1 x 81 mm
- board text removed: "12V"
- board text removed: "3V3"
- board text removed: "CAN_L CAN_H"
