File: pcb/espio.kicad_pcb (KiCad board)
At the start: 2 copper layers, 77.1 x 81 mm, 85 parts, among them J1 Conn_Dbg_Header, J2 Conn_01x07, J3 Conn_01x08, J4 Conn_01x01, J5 Conn_01x08, J6 Conn_01x08, Q1 BC817, Q10 BC817, Q11 BC817, Q12 BC817, Q13 BC817, Q15 BC817, Q16 BC817, Q2 IRLML6402, Q3 BC817, Q4 IRLML6402, Q5 BC817, Q6 IRLML6402, Q7 BC817, Q8 IRLML6402, Q9 BC817, U1 MCP2562-E-SN, U5 LF50CPT-TR, U6 K776180WR-1

Commit message: major work
Parts:
- removed C1, C2, C4: 0.1uF, Capacitor_SMD:C_0603_1608Metric
- removed C3: RVT2A2R2M0605_C335981, lcsc:CAP-SMD_BD6.3-L6.6-W6.6-FD
- removed D1, D3, D4, D5, D6: 1N5819HW-7-F, lcsc:SOD-123_L2.7-W1.6-LS3.7-RD
- removed D2: BZV55C15_C545332, lcsc:SOD-80_L3.5-W1.5-RD
- removed F1, F2, F3, F4: 1812L110/33MR, lcsc:F1812
- removed F5: 1812L050/30PR, lcsc:F1812
- removed J1: Conn_Dbg_Header, Connector_PinHeader_2.54mm:PinHeader_1x02_P2.54mm_Vertical
- removed J2: Conn_01x07, Connector_PinSocket_2.54mm:PinSocket_1x06_P2.54mm_Vertical
- removed J3, J5: Conn_01x08, Connector_PinSocket_2.54mm:PinSocket_1x08_P2.54mm_Vertical
- removed J4: Conn_01x01, Connector_PinHeader_2.54mm:PinHeader_1x01_P2.54mm_Vertical
- removed J6: Conn_01x08, Connector_PinSocket_2.54mm:PinSocket_1x04_P2.54mm_Vertical
- removed JP1, JP3: Jumper_2_Open, Jumper:SolderJumper-2_P1.3mm_Open_Pad1.0x1.5mm
- removed JP2: VCC_as_Pin_8, Jumper:SolderJumper-2_P1.3mm_Open_Pad1.0x1.5mm
- removed LED1, LED2, LED3, LED4, LED5: 0805G (Green), lcsc:LED0805-R-RD
- removed Q1, Q10, Q11, Q12, Q13, Q15, Q16, Q3, Q5, Q7, Q9: BC817, Package_TO_SOT_SMD:SOT-23
- removed Q2, Q4, Q6, Q8: IRLML6402, Package_TO_SOT_SMD:SOT-23
- removed R1, R18, R19, R20, R3: 1k, Resistor_SMD:R_0603_1608Metric
- removed R10, R11, R8, R9: DNP, Resistor_THT:R_Axial_DIN0207_L6.3mm_D2.5mm_P7.62mm_Horizontal
- removed R12, R14, R21, R23, R25, R27, R33, R35: 3k, Resistor_SMD:R_0603_1608Metric
- removed R13, R16, R37, R38: 2k4, Resistor_SMD:R_0603_1608Metric
- removed R15, R17, R22, R24, R26, R28, R34, R36: 750R, Resistor_SMD:R_0603_1608Metric
- removed R2: 4k, Resistor_SMD:R_0603_1608Metric
- removed R29, R30, R31, R32: 10k, Resistor_SMD:R_0603_1608Metric
- removed R39: 470, Resistor_SMD:R_0603_1608Metric
- removed R63: 120R, Resistor_SMD:R_0603_1608Metric
- removed U1: MCP2562-E-SN, Package_SO:SOIC-8_3.9x4.9mm_P1.27mm
- removed U5: LF50CPT-TR, lcsc:PPAK-5_L6.5-W6.1-P1.27-LS10.0-TL
Connections:
- net ABS_INPUT_VR_1 renamed DIRECT_IN_7
- U2 pad 10: /Spannungsteiler7/IN_MEAS -> /v_div8/IN_MEAS
- U2 pad 11: /Spannungsteiler6/IN_MEAS -> DIRECT_IN_1
- U2 pad 12: ABS_INPUT_HR_2 -> DIRECT_IN_2
- U2 pad 13: ABS_INPUT_HR_1 -> DIRECT_IN_3
- U2 pad 14: ABS_INPUT_HL_2 -> DIRECT_IN_4
- U2 pad 15: ABS_INPUT_VR_2 -> DIRECT_IN_5
- U2 pad 16: ABS_INPUT_HL_1 -> DIRECT_IN_6
- U2 pad 18: ABS_INPUT_VL_2 -> DIRECT_IN_8
- U2 pad 19: ABS_INPUT_VL_1 -> DIRECT_IN_9
- U2 pad 3: /Spannungsteiler8/IN_MEAS -> /v_div1/IN_MEAS
- U2 pad 4: /Spannungsteiler1/IN_MEAS -> /v_div2/IN_MEAS
- U2 pad 5: /Spannungsteiler3/IN_MEAS -> /v_div3/IN_MEAS
- U2 pad 6: /Spannungsteiler2/IN_MEAS -> /v_div4/IN_MEAS
- U2 pad 7: /Spannungsteiler4/IN_MEAS -> /v_div5/IN_MEAS
- U2 pad 8: /Spannungsteiler5/IN_MEAS -> /v_div6/IN_MEAS
- U2 pad 9: DIRECT_IN_1 -> /v_div7/IN_MEAS
- U3 pad 10: Net-(J2-Pin_3) -> /pulldown3/IN
- U3 pad 11: Net-(J2-Pin_4) -> /pulldown4/IN
- U3 pad 12: Net-(J2-Pin_5) -> /pulldown5/IN
- U3 pad 13: Net-(J2-Pin_6) -> /pulldown6/IN
- U3 pad 14: /SwitchingNode4/SN_IN -> /powernode4/SN_IN
- U3 pad 15: /SwitchingNode3/SN_IN -> /powernode3/SN_IN
- U3 pad 16: I2C0_SDA -> /powernode2/SN_IN
- U3 pad 17: I2C0_SCL -> /powernode1/SN_IN
- U3 pad 18: /SwitchingNode2/SN_IN -> I2C0_SDA
- U3 pad 19: /SwitchingNode1/SN_IN -> I2C0_SCL
- U3 pad 5: Net-(J2-Pin_1) -> /pulldown1/IN
- U3 pad 8: Net-(J2-Pin_2) -> /pulldown2/IN
- U6 pad 10: /10_12V_OUT -> 12V_OUT_2
- U6 pad 11: /11_12V_OUT -> 12V_OUT_3
- U6 pad 12: /12_12V_OUT -> 12V_OUT_4
- U6 pad 18: ABS_INPUT_HL_2 -> DIRECT_IN_9
- U6 pad 19: ABS_INPUT_HL_1 -> DIRECT_IN_8
- U6 pad 2: I_6 -> I_5
- U6 pad 26: I_8 -> I_6
- U6 pad 27: I_9 -> I_7
- U6 pad 28: I_10 -> I_8
- U6 pad 29: ABS_INPUT_HR_2 -> DIRECT_IN_6
- U6 pad 3: /3_PULL_DOWN -> PULLDOWN_1
- U6 pad 30: ABS_INPUT_HR_1 -> DIRECT_IN_5
- U6 pad 31: ABS_INPUT_VR_2 -> DIRECT_IN_4
- U6 pad 32: ABS_INPUT_VL_1 -> DIRECT_IN_3
- U6 pad 33: ABS_INPUT_VL_2 -> DIRECT_IN_2
- U6 pad 4: /4_PULL_DOWN -> PULLDOWN_2
- U6 pad 5: /5_PULL_DOWN -> PULLDOWN_3
- U6 pad 6: /6_PULL_DOWN -> PULLDOWN_4
- U6 pad 7: /7_PULL_DOWN -> PULLDOWN_5
- U6 pad 8: /8_PULL_DOWN -> PULLDOWN_6
- U6 pad 9: /9_12V_OUT -> 12V_OUT_1
Routing:
- net +5V: track 31.4 -> 0.00 mm
- net +12V: track 27.7 -> 0.00 mm
- net Net-(JP3-B): track 15.3 -> 0.00 mm
- net CAN_H: track 7.88 -> 0.00 mm
- net CAN_L: track 5.95 -> 0.00 mm
- net GND: track 3.13 -> 0.00 mm
- net Net-(D2-A): track 2.69 -> 0.00 mm
- net Net-(JP1-B): track 2.48 -> 0.00 mm
- net Net-(Q16-E): track 2.00 -> 0.00 mm
- net +3V3: track 1.97 -> 0.00 mm
- net Net-(LED5-A): track 1.93 -> 0.00 mm
- removed copper zone on B.Cu, net +12V
Other:
- board text removed: "120R"
- board text removed: "GND"
- board text removed: "Permanent_On"
