File: pcb/powernode.kicad_sch (KiCad schematic)
At the start: 11 parts, among them Q2 2SC1623 300-400, Q4 IRLML6402

Commit message: edit pulldown
Changed lines of the file:
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@@
-	)
-	(junction
-		(at 147.32 83.82)
-		(diameter 0)
-		(color 0 0 0 0)
 	)
 	(junction
@@
 		)
 		(stroke
-			(width 0)
-			(type default)
-		)
-	)
-	(wire
-		(pts
-			(xy 138.43 83.82) (xy 147.32 83.82)
-		)
-		(stroke
