File: pcb/spannungsteiler.kicad_sch (KiCad schematic)
At the start: 2 parts

Commit message: fixed the dumb schematic
Other:
- note added: "Kondensator?"
Changed lines of the file:
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@@
 	(generator_version "9.0")
 	(paper "A4")
+	(text "Kondensator?"
+		(exclude_from_sim no)
+		(at 106.68 93.98 0)
+		(effects
+			(font
+				(size 1.27 1.27)
+			)
+		)
+	)
+	(junction
+		(at 120.65 97.79)
+		(diameter 0)
+		(color 0 0 0 0)
+	)
 	(junction
 		(at 120.65 86.36)
@@
 	(wire
 		(pts
-			(xy 120.65 99.06) (xy 120.65 95.25)
+			(xy 120.65 99.06) (xy 120.65 97.79)
 		)
 		(stroke
@@
 		(pts
 			(xy 120.65 82.55) (xy 120.65 86.36)
+		)
+		(stroke
+			(width 0)
+			(type default)
+		)
+	)
+	(wire
+		(pts
+			(xy 106.68 86.36) (xy 106.68 91.44)
+		)
+		(stroke
+			(width 0)
+			(type default)
+		)
+	)
+	(wire
+		(pts
+			(xy 106.68 97.79) (xy 120.65 97.79)
 		)
 		(stroke
@@
 		)
 		(stroke
+			(width 0)
+			(type default)
+		)
+	)
+	(wire
+		(pts
+			(xy 120.65 86.36) (xy 106.68 86.36)
+		)
+		(stroke
+			(width 0)
+			(type default)
+		)
+	)
+	(wire
+		(pts
+			(xy 120.65 97.79) (xy 120.65 95.25)
+		)
+		(stroke
+			(width 0)
+			(type default)
+		)
+	)
+	(wire
+		(pts
+			(xy 106.68 95.25) (xy 106.68 97.79)
+		)
+		(stroke

Commit message: major work
Parts:
- renumbered R12 to R14, R17 to R15
Changed lines of the file:
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@@
 		(on_board yes)
 		(dnp no)
-		(property "Reference" "R12"
+		(property "Reference" "R14"
 			(at 119.38 76.2 90)
 			(effects
@@
 		)
 		(property "Value" "3k"
-			(at 120.65 81.28 90)
+			(at 120.65 80.264 90)
 			(effects
 				(font
@@
 		(instances
 			(project "espio"
-				(path "/b4b62778-ee22-463e-ba5d-5da015edb128/7c02ff32-7f45-4779-bda1-df17b806787c"
+				(path "/b4b62778-ee22-463e-ba5d-5da015edb128/210f7e6f-ab19-4145-9402-ce13a28f3acc"
+					(reference "R12")
+					(unit 1)
+				)
+				(path "/b4b62778-ee22-463e-ba5d-5da015edb128/5cfb3e15-3011-460b-8df1-a63b2e3a4420"
+					(reference "R35")
+					(unit 1)
+				)
+				(path "/b4b62778-ee22-463e-ba5d-5da015edb128/a4c53919-bb0e-4d9c-9e6a-dc9a4c4b3a35"
+					(reference "R23")
+					(unit 1)
+				)
+				(path "/b4b62778-ee22-463e-ba5d-5da015edb128/abb4e55a-5c59-4a44-97d5-a085a39dce1d"
+					(reference "R27")
+					(unit 1)
+				)
+				(path "/b4b62778-ee22-463e-ba5d-5da015edb128/b74ef4bc-ea8f-4137-b14f-72ea8a7b76e7"
+					(reference "R25")
+					(unit 1)
+				)
+				(path "/b4b62778-ee22-463e-ba5d-5da015edb128/da5b8548-51a2-4008-ae18-2aef51f98485"
 					(reference "R33")
 					(unit 1)
 				)
-				(path "/b4b62778-ee22-463e-ba5d-5da015edb128/9951c11d-3347-4ddd-848f-60f8e40d62bf"
-					(reference "R12")
-					(unit 1)
-				)
-				(path "/b4b62778-ee22-463e-ba5d-5da015edb128/9fbcdd6f-7683-42a0-8e27-28d1be0e1488"
-					(reference "R35")
-					(unit 1)
-				)
-				(path "/b4b62778-ee22-463e-ba5d-5da015edb128/c9de4cad-5bdd-4b0b-a4e5-53fd8ec2ca1e"
+				(path "/b4b62778-ee22-463e-ba5d-5da015edb128/e57b8cdf-3f96-436e-9519-20254e22b287"
 					(reference "R21")
-					(unit 1)
-				)
-				(path "/b4b62778-ee22-463e-ba5d-5da015edb128/cb2509ee-5c67-41ae-a1d3-21ee1dfa5bf2"
-					(reference "R27")
-					(unit 1)
-				)
-				(path "/b4b62778-ee22-463e-ba5d-5da015edb128/d599d020-d1ba-4fdf-8176-2d51b64b0e6a"
-					(reference "R25")
-					(unit 1)
-				)
-				(path "/b4b62778-ee22-463e-ba5d-5da015edb128/e53e8619-f807-4da0-899d-5834b6bfa097"
-					(reference "R23")
 					(unit 1)
 				)
@@
 		(dnp no)
 		(fields_autoplaced yes)
-		(property "Reference" "#PWR024"
+		(property "Reference" "#PWR038"
 			(at 120.65 105.41 0)
 			(effects
@@
 		(instances
 			(project "espio"
-				(path "/b4b62778-ee22-463e-ba5d-5da015edb128/7c02ff32-7f45-4779-bda1-df17b806787c"
+				(path "/b4b62778-ee22-463e-ba5d-5da015edb128/210f7e6f-ab19-4145-9402-ce13a28f3acc"
+					(reference "#PWR024")
+					(unit 1)
+				)
+				(path "/b4b62778-ee22-463e-ba5d-5da015edb128/5cfb3e15-3011-460b-8df1-a63b2e3a4420"
+					(reference "#PWR037")
+					(unit 1)
+				)
+				(path "/b4b62778-ee22-463e-ba5d-5da015edb128/a4c53919-bb0e-4d9c-9e6a-dc9a4c4b3a35"
+					(reference "#PWR026")
+					(unit 1)
+				)
+				(path "/b4b62778-ee22-463e-ba5d-5da015edb128/abb4e55a-5c59-4a44-97d5-a085a39dce1d"
+					(reference "#PWR034")
+					(unit 1)
+				)
+				(path "/b4b62778-ee22-463e-ba5d-5da015edb128/b74ef4bc-ea8f-4137-b14f-72ea8a7b76e7"
+					(reference "#PWR027")
+					(unit 1)
+				)
+				(path "/b4b62778-ee22-463e-ba5d-5da015edb128/da5b8548-51a2-4008-ae18-2aef51f98485"
 					(reference "#PWR036")
 					(unit 1)
 				)
-				(path "/b4b62778-ee22-463e-ba5d-5da015edb128/9951c11d-3347-4ddd-848f-60f8e40d62bf"
-					(reference "#PWR024")
-					(unit 1)
-				)
-				(path "/b4b62778-ee22-463e-ba5d-5da015edb128/9fbcdd6f-7683-42a0-8e27-28d1be0e1488"
-					(reference "#PWR037")
-					(unit 1)
-				)
-				(path "/b4b62778-ee22-463e-ba5d-5da015edb128/c9de4cad-5bdd-4b0b-a4e5-53fd8ec2ca1e"
+				(path "/b4b62778-ee22-463e-ba5d-5da015edb128/e57b8cdf-3f96-436e-9519-20254e22b287"
 					(reference "#PWR025")
-					(unit 1)
-				)
-				(path "/b4b62778-ee22-463e-ba5d-5da015edb128/cb2509ee-5c67-41ae-a1d3-21ee1dfa5bf2"
-					(reference "#PWR034")
-					(unit 1)
-				)
-				(path "/b4b62778-ee22-463e-ba5d-5da015edb128/d599d020-d1ba-4fdf-8176-2d51b64b0e6a"
-					(reference "#PWR027")
-					(unit 1)
-				)
-				(path "/b4b62778-ee22-463e-ba5d-5da015edb128/e53e8619-f807-4da0-899d-5834b6bfa097"
-					(reference "#PWR026")
 					(unit 1)
 				)
@@
 		(on_board yes)
 		(dnp no)
-		(property "Reference" "R17"
+		(property "Reference" "R15"
 			(at 117.856 93.218 90)
 			(effects
@@
 		(instances
 			(project "espio"
-				(path "/b4b62778-ee22-463e-ba5d-5da015edb128/7c02ff32-7f45-4779-bda1-df17b806787c"
+				(path "/b4b62778-ee22-463e-ba5d-5da015edb128/210f7e6f-ab19-4145-9402-ce13a28f3acc"
+					(reference "R17")
+					(unit 1)
+				)
+				(path "/b4b62778-ee22-463e-ba5d-5da015edb128/5cfb3e15-3011-460b-8df1-a63b2e3a4420"
+					(reference "R36")
+					(unit 1)
+				)
+				(path "/b4b62778-ee22-463e-ba5d-5da015edb128/a4c53919-bb0e-4d9c-9e6a-dc9a4c4b3a35"
+					(reference "R24")
+					(unit 1)
+				)
+				(path "/b4b62778-ee22-463e-ba5d-5da015edb128/abb4e55a-5c59-4a44-97d5-a085a39dce1d"
+					(reference "R28")
+					(unit 1)
+				)
+				(path "/b4b62778-ee22-463e-ba5d-5da015edb128/b74ef4bc-ea8f-4137-b14f-72ea8a7b76e7"
+					(reference "R26")
+					(unit 1)
+				)
+				(path "/b4b62778-ee22-463e-ba5d-5da015edb128/da5b8548-51a2-4008-ae18-2aef51f98485"
 					(reference "R34")
 					(unit 1)
 				)
-				(path "/b4b62778-ee22-463e-ba5d-5da015edb128/9951c11d-3347-4ddd-848f-60f8e40d62bf"
-					(reference "R17")
-					(unit 1)
-				)
-				(path "/b4b62778-ee22-463e-ba5d-5da015edb128/9fbcdd6f-7683-42a0-8e27-28d1be0e1488"
-					(reference "R36")
-					(unit 1)
-				)
-				(path "/b4b62778-ee22-463e-ba5d-5da015edb128/c9de4cad-5bdd-4b0b-a4e5-53fd8ec2ca1e"
+				(path "/b4b62778-ee22-463e-ba5d-5da015edb128/e57b8cdf-3f96-436e-9519-20254e22b287"
 					(reference "R22")
 					(unit 1)
 				)
-				(path "/b4b62778-ee22-463e-ba5d-5da015edb128/cb2509ee-5c67-41ae-a1d3-21ee1dfa5bf2"
-					(reference "R28")
-					(unit 1)
-				)
-				(path "/b4b62778-ee22-463e-ba5d-5da015edb128/d599d020-d1ba-4fdf-8176-2d51b64b0e6a"
-					(reference "R26")
-					(unit 1)
-				)
-				(path "/b4b62778-ee22-463e-ba5d-5da015edb128/e53e8619-f807-4da0-899d-5834b6bfa097"
-					(reference "R24")
-					(unit 1)
-				)
