File: pcb/v2_5/espio.kicad_sch (KiCad schematic)
At the start: 27 parts, among them J1 Conn_Dbg_Header, J2 Conn_01x07, J3 Conn_01x08, J4 Conn_01x01, J5 Conn_01x08, J6 Conn_01x08, Q16 BC817, U1 MCP2562-E-SN, U5 LF50CPT-TR, U6 K776180WR-1

Commit message: added some diodes, fuses etc
Parts:
- removed D6: 1N5819HW-7-F, lcsc:SOD-123_L2.7-W1.6-LS3.7-RD, symbol lcsc:1N5819HW-7-F
- removed F5: 1812L050/30PR, lcsc:F1812, symbol lcsc:1812L050_30PR
- removed LED1: ORH-B36G, lcsc:LED0603-RD, symbol lcsc:ORH-B36G
- removed R44: 1k, Resistor_SMD:R_0603_1608Metric, symbol Device:R
- added LED5: 0805G (Green), lcsc:LED0805-R-RD, symbol lcsc:0805G(Green)
- added Q10, Q11, Q12, Q13, Q15, Q9: BC817, Package_TO_SOT_SMD:SOT-23, symbol Transistor_BJT:BC817
- added R39: 470, Resistor_SMD:R_0603_1608Metric, symbol Device:R
Connections:
- net I_5 is gone; now on net I_6: U6.2
- net +12V: now also C4.1, U5.1 (VIN)
- net +5V: now also R39.1
- net 3_PULL_DOWN: now also Q13.3 (C)
- net 4_PULL_DOWN: now also Q12.3 (C)
- net 5_PULL_DOWN: now also Q15.3 (C)
- net 6_PULL_DOWN: now also Q10.3 (C)
- net 7_PULL_DOWN: now also Q9.3 (C)
- net 8_PULL_DOWN: now also Q11.3 (C)
- net GND: now also LED5.2 (K), Q10.2 (E), Q11.2 (E), Q12.2 (E), Q13.2 (E), Q15.2 (E), Q9.2 (E)
- net I2C0_SCL: now also U3.17 (42); no longer U3.19 (1)
- net I2C0_SDA: now also U3.16 (41); no longer U3.18 (2)
- net I_6: no longer U6.26
- net I_8: now also U6.26; no longer U6.28
- net SwitchingNode1/SN_IN: now also U3.19 (1); no longer U3.17 (42)
- net SwitchingNode2/SN_IN: now also U3.18 (2); no longer U3.16 (41)
- net DIRECT_IN_1 renamed OUT_1
- net I_7 renamed I_9
- net pulldown1/IN: no longer names the net of J2.1 (Pin_1), U3.5 (21)
- net pulldown1/IN: now also Q13.1 (B)
- net pulldown2/IN: no longer names the net of J2.2 (Pin_2), U3.8 (45)
- net pulldown2/IN: now also Q12.1 (B)
- net pulldown3/IN: no longer names the net of J2.3 (Pin_3), U3.10 (35)
- net pulldown3/IN: now also Q15.1 (B)
- net pulldown4/IN: no longer names the net of J2.4 (Pin_4), U3.11 (36)
- net pulldown4/IN: now also Q10.1 (B)
- net pulldown5/IN: no longer names the net of J2.5 (Pin_5), U3.12 (37)
- net pulldown5/IN: now also Q9.1 (B)
- net pulldown6/IN: no longer names the net of J2.6 (Pin_6), U3.13 (38)
- net pulldown6/IN: now also Q11.1 (B)
- new net: LED5.1 (A), R39.2
- new net I_10: U6.28
Other:
- removed sheet pulldown1
- removed sheet pulldown2
- removed sheet pulldown3
- removed sheet pulldown4
- removed sheet pulldown5
- removed sheet pulldown6
- sheet SwitchingNode1 ports: added none; removed POWER
- sheet SwitchingNode2 ports: added none; removed POWER
- sheet SwitchingNode3 ports: added none; removed POWER
- sheet SwitchingNode4 ports: added none; removed POWER
- moved on the sheet: C3, C4, D2, J2, J3, J4, J5, J6, JP2, JP3, Q16, R2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
