File: pcb/v2_6/espio.kicad_pcb (KiCad board)
At the start: 2 copper layers, 77.1 x 82.9 mm, 155 parts, among them J1 Conn_Dbg_Header, J2 Conn_01x08, J3 Conn_01x09, J4 Conn_01x01, J5 Conn_01x08, J6 Conn_01x08, Q1 2SC1623 300-400, Q10 2SC1623 300-400, Q11 IRLML6402, Q12 2SC1623 300-400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

Commit message: Refactor, fix external LED conflict
Parts:
- moved J5 4.48 mm to (94.8, 95.6)
- moved R33 3.92 mm to (99.1, 109.7)
- moved R12 3.92 mm to (99.0, 97.0)
- moved R14 3.92 mm to (99.0, 94.5)
- moved R21 3.92 mm to (99.0, 99.6)
- moved R23 3.92 mm to (99.0, 102.1)
- moved R25 3.92 mm to (99.0, 104.6)
- moved R27 3.92 mm to (99.0, 107.2)
- moved R35 3.77 mm to (99.1, 111.5)
Routing:
- net I_1: track 73.7 -> 76.9 mm
- net I_8: track 59.1 -> 61.9 mm
- net I_3: track 70.6 -> 73.3 mm
- net I_6: track 61.6 -> 64.2 mm
- net I_2: track 68.7 -> 71.3 mm
- net I_4: track 64.6 -> 67.1 mm
- net I_7: track 63.7 -> 66.2 mm
- net I_5: track 66.7 -> 69.1 mm
- net /v_div8/IN_MEAS: track 9.56 -> 11.5 mm
- net /v_div7/IN_MEAS: track 9.55 -> 10.9 mm
- net /v_div6/IN_MEAS: track 9.62 -> 10.9 mm
- net /v_div5/IN_MEAS: track 9.56 -> 10.8 mm
- net /v_div4/IN_MEAS: track 9.62 -> 10.9 mm
- net /v_div3/IN_MEAS: track 9.68 -> 11.0 mm
- net /v_div2/IN_MEAS: track 9.68 -> 11.0 mm
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